File: hardware/STM32 RF Dongle.sch (KiCad schematic (older format))
At the start: 39 parts, among them J1 USB_B_Micro, J2 SMA, J3 SWD, U1 NRF24L01, U2 XC6206P332MR, U3 USBLC6-2SC6, U4 STM32L432KBUx, Y1 16MHz

Commit message: added image and minor schematic tidy up
Parts:
- U2: symbol Dobbs:XC6206P332MR -> STM32-RF-Dongle-rescue:XC6206P332MR-Dobbs
Changed lines of the file:
@@
 $EndComp
 $Comp
-L Dobbs:XC6206P332MR U2
+L STM32-RF-Dongle-rescue:XC6206P332MR-Dobbs U2
 U 1 1 5FECB991
 P 2550 1400
